File: Rev. 0/Eagle/U64_KB_Ada.brd (EAGLE design)
At the start: 71 x 56 mm, 9 parts, among them J1 PINS_1X20

Commit message: Silk Screen Update
Other:
- board text added: "http://github.com/svenpetersen1965"
Changed lines of the file:
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@@
 <text x="44.45" y="70.00875" size="1.778" layer="48" font="vector" ratio="12">0</text>
 <text x="69.69125" y="20.47875" size="1.27" layer="21" ratio="12" rot="R90">collaboration with @edu_arana</text>
+<text x="63.34125" y="5.3975" size="1.016" layer="21" ratio="12" rot="R90">http://github.com/svenpetersen1965</text>
 </plain>
 <attributes>
