File: Rev. 0/Eagle/U64_KB_Ada.sch (EAGLE design)
At the start: 6 parts, among them J1 PINS_1X20

Commit message: Silk Screen Update
Other:
- note added: "http://github.com/svenpetersen1965"
Changed lines of the file:
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@@
 <text x="347.98" y="22.86" size="2.54" layer="95">Sven Petersen</text>
 <text x="340.36" y="17.78" size="2.54" layer="95">0</text>
+<text x="279.4" y="7.62" size="2.54" layer="95">http://github.com/svenpetersen1965</text>
 </plain>
 <instances>
